File: 02_HW/stm32_target.kicad_sch (KiCad schematic)
At the start: 12 parts, among them J1 glitch, J2 adc_measure, J3 Conn_02x04_Odd_Even, J4 P1, J5 P2, J6 USB_SERIAL, J7 USB_STM32, U1 STM32F103C8Tx, U2 CH340G, U3 TLV76133

Commit message: [WIP] (HW) add labels and signals
Parts:
- removed J5: P2, Connector_PinHeader_2.54mm:PinHeader_2x05_P2.54mm_Vertical, symbol Connector_Generic:Conn_02x05_Odd_Even
- added J5: P1, Connector_PinHeader_2.54mm:PinHeader_2x10_P2.54mm_Vertical, symbol Connector_Generic:Conn_02x10_Odd_Even
- J4: footprint Connector_PinHeader_2.54mm:PinHeader_2x05_P2.54mm_Vertical -> Connector_PinHeader_2.54mm:PinHeader_2x10_P2.54mm_Vertical; symbol Connector_Generic:Conn_02x05_Odd_Even -> Connector_Generic:Conn_02x10_Odd_Even
Connections:
- net +3.3V: now also J4.18 (Pin_18), J5.16 (Pin_16), J5.18 (Pin_18)
- net GND: now also J4.19 (Pin_19), J6.A1 (GND), J6.A12 (GND), J6.B1 (GND), J6.B12 (GND), J6.S1 (SHIELD), J7.A1 (GND), J7.A12 (GND), J7.B1 (GND), J7.B12 (GND), J7.S1 (SHIELD), J5.17 (Pin_17), J5.19 (Pin_19)
- net VBUS: now also J4.20 (Pin_20), J6.A4 (VBUS), J6.A9 (VBUS), J6.B4 (VBUS), J6.B9 (VBUS), J5.20 (Pin_20)
- net PA0: now reaches U1.10 (PA0)
- net PA0: now also J4.1 (Pin_1)
- net PA1: now reaches U1.11 (PA1)
- net PA1: now also J4.2 (Pin_2)
- net PA2: now reaches U1.12 (PA2)
- net PA2: now also J4.3 (Pin_3)
- net PA3: now reaches U1.13 (PA3)
- net PA3: now also J4.4 (Pin_4)
- net PA4: now reaches U1.14 (PA4)
- net PA4: now also J4.5 (Pin_5)
- net PA5: now reaches U1.15 (PA5)
- net PA5: now also J4.6 (Pin_6)
- net PA6: now reaches U1.16 (PA6)
- net PA6: now also J4.7 (Pin_7)
- net PA7: now reaches U1.17 (PA7)
- net PA7: now also J4.8 (Pin_8)
- net PB0: now reaches U1.18 (PB0)
- net PB0: now also J4.9 (Pin_9)
- net PB1: now reaches U1.19 (PB1)
- net PB1: now also J4.10 (Pin_10)
- net PC13: now reaches U1.2 (PC13)
- net PB2: now reaches U1.20 (PB2)
- net PB2: now also J4.11 (Pin_11)
- net PB10: now reaches U1.21 (PB10)
- net PB10: now also J4.12 (Pin_12)
- net PB11: now reaches U1.22 (PB11)
- net PB11: now also J4.13 (Pin_13)
- net PB12: now reaches U1.25 (PB12)
- net PB12: now also J4.14 (Pin_14)
- net PB13: now reaches U1.26 (PB13)
- net PB13: now also J4.15 (Pin_15)
- net PB14: now reaches U1.27 (PB14)
- net PB14: now also J4.16 (Pin_16)
- net PB15: now reaches U1.28 (PB15)
- net PB15: now also J4.17 (Pin_17)
- net PA8: now reaches U1.29 (PA8)
- net PA8: now also J5.1 (Pin_1)
- net OSC32_P: now reaches U1.3 (PC14)
- net PA9: now reaches U1.30 (PA9)
- net PA9: now also J5.2 (Pin_2)
- net PA10: now reaches U1.31 (PA10)
- net PA10: now also J5.3 (Pin_3)
- net PA11: now reaches U1.32 (PA11)
- net PA11: now also J5.4 (Pin_4)
- net PA12: now reaches U1.33 (PA12)
- net PA12: now also J5.5 (Pin_5)
- net PA13: now reaches U1.34 (PA13)
- net PA13: now also J5.6 (Pin_6)
- net PA14: now reaches U1.37 (PA14)
- net PA14: now also J5.7 (Pin_7)
- net PA15: now reaches U1.38 (PA15)
- net PA15: now also J5.8 (Pin_8)
- net PB3: now reaches U1.39 (PB3)
- net PB3: now also J5.9 (Pin_9)
- net OSC32_M: now reaches U1.4 (PC15)
- net PB4: now reaches U1.40 (PB4)
- net PB4: now also J5.10 (Pin_10)
- net PB5: now reaches U1.41 (PB5)
- net PB5: now also J5.11 (Pin_11)
- net PB6: now reaches U1.42 (PB6)
- net PB6: now also J5.12 (Pin_12)
- net PB7: now reaches U1.43 (PB7)
- net PB7: now also J5.13 (Pin_13)
- net BOOT_0: now reaches U1.44 (BOOT0)
- net PB8: now reaches U1.45 (PB8)
- net PB8: now also J5.14 (Pin_14)
- net PB9: now reaches U1.46 (PB9)
- net PB9: now also J5.15 (Pin_15)
- net OSC_P: now reaches U1.5 (PD0)
- net OSC_M: now reaches U1.6 (PD1)
- net RST: now reaches U1.7 (NRST)
- net D_P: now reaches J7.A6 (D+)
- net D_P: now also J7.B6 (D+)
- net D_M: now reaches J7.A7 (D-)
- net D_M: now also J7.B7 (D-)
- net CC1: now reaches J6.A5 (CC1)
- net D_UART_P: now reaches J6.A6 (D+)
- net D_UART_P: now also J6.B6 (D+)
- net D_UART_M: now reaches J6.A7 (D-)
- net D_UART_M: now also J6.B7 (D-)
- net CC2: now reaches J6.B5 (CC2)
- no-connect marks 0 -> 3
